Commit message: Fix analytical transform mismatch

File: lab7/urdf/rtr_manipulator.xacro (robot description, xacro)
@@ -94,5 +94,5 @@
     <child link="link_forearm"/>
     <origin xyz="${l2} 0 0" rpy="0 0 0"/>
-    <axis xyz="0 1 0"/>
+    <axis xyz="0 -1 0"/>
     <limit lower="-3.14159" upper="3.14159" effort="100" velocity="1.0"/>
   </joint>

Commit message: Refine Xacro model

File: lab7/urdf/rtr_manipulator.xacro (robot description, xacro)
@@ -1,21 +1,114 @@
 <?xml version="1.0"?>
 <robot xmlns:xacro="http://www.ros.org/wiki/xacro" name="rtr_manipulator">
-  <!-- RTR: Revolute (base yaw) – Prismatic (vertical) – Revolute (elbow). -->
+  <!-- ================= PARAMETERS ================= -->
   <xacro:property name="l2" value="0.9"/>
   <xacro:property name="l3" value="1.0"/>
   <xacro:property name="width" value="0.08"/>
+  <xacro:property name="base_radius" value="0.12"/>
+  <xacro:property name="base_height" value="0.10"/>
+  <xacro:property name="yaw_radius" value="0.06"/>
+  <xacro:property name="yaw_height" value="0.30"/>
+  <xacro:property name="tool_radius" value="0.03"/>
+  <xacro:property name="tool_length" value="0.12"/>
+  <!-- ================= MATERIALS ================= -->
   <material name="blue"><color rgba="0 0 1 1"/></material>
   <material name="red"><color rgba="1 0 0 1"/></material>
   <material name="green"><color rgba="0 1 0 1"/></material>
   <material name="grey"><color rgba="0.7 0.7 0.7 1"/></material>
+  <!-- ================= MACROS ================= -->
+  <xacro:macro name="box_link" params="name size_x size_y size_z origin_x origin_y origin_z mass material_name">
+    <link name="${name}">
+      <inertial>
+        <origin xyz="${origin_x} ${origin_y} ${origin_z}" rpy="0 0 0"/>
+        <mass value="${mass}"/>
+        <inertia ixx="0.1" ixy="0" ixz="0" iyy="0.1" iyz="0" izz="0.1"/>
+      </inertial>
+      <visual>
+        <origin xyz="${origin_x} ${origin_y} ${origin_z}" rpy="0 0 0"/>
+        <geometry>
+          <box size="${size_x} ${size_y} ${size_z}"/>
+        </geometry>
+        <material name="${material_name}"/>
+      </visual>
+      <collision>
+        <origin xyz="${origin_x} ${origin_y} ${origin_z}" rpy="0 0 0"/>
+        <geometry>
+          <box size="${size_x} ${size_y} ${size_z}"/>
+        </geometry>
+      </collision>
+    </link>
+  </xacro:macro>
+  <xacro:macro name="cylinder_link" params="name radius length origin_x origin_y origin_z mass material_name">
+    <link name="${name}">
+      <inertial>
+        <origin xyz="${origin_x} ${origin_y} ${origin_z}" rpy="0 0 0"/>
+        <mass value="${mass}"/>
+        <inertia ixx="0.05" ixy="0" ixz="0" iyy="0.05" iyz="0" izz="0.05"/>
+      </inertial>
+      <visual>
+        <origin xyz="${origin_x} ${origin_y} ${origin_z}" rpy="0 0 0"/>
+        <geometry>
+          <cylinder radius="${radius}" length="${length}"/>
+        </geometry>
+        <material name="${material_name}"/>
+      </visual>
+      <collision>
+        <origin xyz="${origin_x} ${origin_y} ${origin_z}" rpy="0 0 0"/>
+        <geometry>
+          <cylinder radius="${radius}" length="${length}"/>
+        </geometry>
+      </collision>
+    </link>
+  </xacro:macro>
+  <!-- ================= LINKS ================= -->
   <link name="world"/>
-  <!-- Origins chosen so joint variables match the paper FK (no extra vertical offset in theta_2). -->
-  <link name="base_link">
+  <xacro:cylinder_link
+    name="base_link"
+    radius="${base_radius}"
+    length="${base_height}"
+    origin_x="0" origin_y="0" origin_z="${base_height/2}"
+    mass="5"
+    material_name="grey"/>
+  <xacro:cylinder_link
+    name="link_yaw"
+    radius="${yaw_radius}"
+    length="${yaw_height}"
+    origin_x="0" origin_y="0" origin_z="${yaw_height/2}"
+    mass="2"
+    material_name="blue"/>
+  <xacro:box_link
+    name="link_carriage"
+    size_x="${width}" size_y="${width}" size_z="${width}"
+    origin_x="0" origin_y="0" origin_z="0"
+    mass="1"
+    material_name="green"/>
+  <xacro:box_link
+    name="link_upper"
+    size_x="${l2}" size_y="${width}" size_z="${width}"
+    origin_x="${l2/2}" origin_y="0" origin_z="0"
+    mass="10"
+    material_name="red"/>
+  <xacro:box_link
+    name="link_forearm"
+    size_x="${l3}" size_y="${width}" size_z="${width}"
+    origin_x="${l3/2}" origin_y="0" origin_z="0"
+    mass="10"
+    material_name="blue"/>
+  <link name="tool0">
     <visual>
-      <origin xyz="0 0 0.05" rpy="0 0 0"/>
-      <geometry><cylinder radius="0.12" length="0.1"/></geometry>
-      <material name="grey"/>
+      <origin xyz="${tool_length/2} 0 0" rpy="0 1.5708 0"/>
+      <geometry>
+        <cylinder radius="${tool_radius}" length="${tool_length}"/>
+      </geometry>
+      <material name="green"/>
     </visual>
+    <collision>
+      <origin xyz="${tool_length/2} 0 0" rpy="0 1.5708 0"/>
+      <geometry>
+        <cylinder radius="${tool_radius}" length="${tool_length}"/>
+      </geometry>
+    </collision>
   </link>
+  <!-- ================= JOINTS ================= -->
   <joint name="world_to_base" type="fixed">
     <parent link="world"/>
@@ -23,16 +116,4 @@
     <origin xyz="0 0 0" rpy="0 0 0"/>
   </joint>
-  <link name="link_yaw">
-    <inertial>
-      <origin xyz="0 0 0" rpy="0 0 0"/>
-      <mass value="1"/>
-      <inertia ixx="0.01" ixy="0" ixz="0" iyy="0.01" iyz="0" izz="0.01"/>
-    </inertial>
-    <visual>
-      <origin xyz="0 0 0.15" rpy="0 0 0"/>
-      <geometry><cylinder radius="0.06" length="0.3"/></geometry>
-      <material name="blue"/>
-    </visual>
-  </link>
   <joint name="joint_theta1" type="revolute">
     <parent link="base_link"/>
@@ -42,16 +123,4 @@
     <limit lower="-3.14159" upper="3.14159" effort="100" velocity="1.0"/>
   </joint>
-  <link name="link_carriage">
-    <inertial>
-      <origin xyz="0 0 0" rpy="0 0 0"/>
-      <mass value="1"/>
-      <inertia ixx="0.01" ixy="0" ixz="0" iyy="0.01" iyz="0" izz="0.01"/>
-    </inertial>
-    <visual>
-      <origin xyz="0 0 0" rpy="0 0 0"/>
-      <geometry><box size="${width} ${width} ${width}"/></geometry>
-      <material name="green"/>
-    </visual>
-  </link>
   <joint name="joint_theta2" type="prismatic">
     <parent link="link_yaw"/>
@@ -61,16 +130,4 @@
     <limit lower="0.0" upper="2.0" effort="200" velocity="0.25"/>
   </joint>
-  <link name="link_upper">
-    <inertial>
-      <origin xyz="${l2/2} 0 0" rpy="0 0 0"/>
-      <mass value="20"/>
-      <inertia ixx="0.1" ixy="0" ixz="0" iyy="1" iyz="0" izz="1"/>
-    </inertial>
-    <visual>
-      <origin xyz="${l2/2} 0 0" rpy="0 0 0"/>
-      <geometry><box size="${l2} ${width} ${width}"/></geometry>
-      <material name="red"/>
-    </visual>
-  </link>
   <joint name="fixed_carriage_upper" type="fixed">
     <parent link="link_carriage"/>
@@ -78,16 +135,4 @@
     <origin xyz="0 0 0" rpy="0 0 0"/>
   </joint>
-  <link name="link_forearm">
-    <inertial>
-      <origin xyz="${l3/2} 0 0" rpy="0 0 0"/>
-      <mass value="20"/>
-      <inertia ixx="0.1" ixy="0" ixz="0" iyy="1" iyz="0" izz="1"/>
-    </inertial>
-    <visual>
-      <origin xyz="${l3/2} 0 0" rpy="0 0 0"/>
-      <geometry><box size="${l3} ${width} ${width}"/></geometry>
-      <material name="blue"/>
-    </visual>
-  </link>
   <joint name="joint_theta3" type="revolute">
     <parent link="link_upper"/>
@@ -97,5 +142,4 @@
     <limit lower="-3.14159" upper="3.14159" effort="100" velocity="1.0"/>
   </joint>
-  <link name="tool0"/>
   <joint name="wrist_to_tool0" type="fixed">
     <parent link="link_forearm"/>
@@ -103,5 +147,5 @@
     <origin xyz="${l3} 0 0" rpy="0 0 0"/>
   </joint>
-  <!-- Ignored by joint_state_publisher_gui / classic chain; required for ros2_control bringup. -->
+  <!-- ================= ROS2 CONTROL ================= -->
   <ros2_control name="RTRMock" type="system">
     <hardware>
